Commit message: morning push

File: description/ros2_control/cx165l.ros2_control.xacro (robot description, xacro)
@@ -1,5 +1,5 @@
 <?xml version="1.0"?>
 <robot xmlns:xacro="http://www.ros.org/wiki/xacro">
-  <xacro:macro name="cx110l_ros2_control" params="name">
+  <xacro:macro name="cx165l_ros2_control" params="name">
     <ros2_control name="${name}" type="system">
       <hardware>
@@ -12,6 +12,6 @@
       <joint name="joint_1">
         <command_interface name="position">
-          <param name="min">${radians(0)}</param>
-          <param name="max">${radians(90)}</param>
+          <param name="min">${radians(-160)}</param>
+          <param name="max">${radians(160)}</param>
         </command_interface>
         <command_interface name="velocity">
@@ -26,6 +26,6 @@
       <joint name="joint_2">
         <command_interface name="position">
-          <param name="min">${radians(-80)}</param>
-          <param name="max">${radians(36)}</param>
+          <param name="min">${radians(-60)}</param>
+          <param name="max">${radians(80)}</param>
         </command_interface>
         <command_interface name="velocity">
@@ -41,5 +41,5 @@
         <command_interface name="position">
           <param name="min">${radians(-75)}</param>
-          <param name="max">${radians(0)}</param>
+          <param name="max">${radians(95)}</param>
         </command_interface>
         <command_interface name="velocity">

File: description/urdf/cx165l.urdf.xacro (robot description, xacro)
@@ -1,6 +1,6 @@
 <?xml version="1.0"?>
-<robot xmlns:xacro="http://wiki.ros.org/xacro" name="cx110l">
-  <xacro:property name="robot_name" value="cx110l"/>
-  <!-- Import cx110l macro -->
+<robot xmlns:xacro="http://wiki.ros.org/xacro" name="cx165l">
+  <xacro:property name="robot_name" value="cx165l"/>
+  <!-- Import cx165l macro -->
   <xacro:include filename="$(find khi2cpp_hw_description)/${robot_name}/urdf/${robot_name}_description.urdf.xacro"/>
   <!-- create link fixed to the "world" -->
@@ -8,7 +8,7 @@
   <!-- Import Lab Robot Cell -->
   <xacro:include filename="$(find khi2cpp_hw)/urdf/isu_lab.xacro" />
-  <xacro:cx110l_description/>
+  <xacro:cx165l_description/>
   <!-- Import cx110l ros2_control description -->
   <xacro:include filename="$(find khi2cpp_hw)/ros2_control/${robot_name}.ros2_control.xacro" />
-  <xacro:cx110l_ros2_control name="${robot_name}"/>
+  <xacro:cx165l_ros2_control name="${robot_name}"/>
 </robot>

File: description/urdf/isu_lab.xacro (robot description, xacro)
@@ -8,11 +8,11 @@
       </inertial>
     </xacro:macro>
-    <joint name="base_plate_to_world" type="fixed">
-        <parent link="world"/>
-        <child link="base_plate"/>
-        <origin rpy="0 0 0" xyz="0 0 0"/>
-    </joint>
     <!-- Lab Environment -->
-     <link name="base_plate">
+    <joint name="cx165l_baseplate" type="fixed">
+        <parent link="world"/>
+        <child link="base_plate_cx165l"/>
+        <origin rpy="0 0 0" xyz="0 0 0"/>
+    </joint>
+    <link name="base_plate_cx165l">
         <parent link="world"/>
         <visual>
@@ -39,4 +39,34 @@
         <xacro:default_inertial mass="1"/>
     </link>
+    <joint name="cx110l_baseplate" type="fixed">
+        <parent link="world"/>
+        <child link="base_plate_cx110l"/>
+        <origin rpy="0 0 0" xyz="-5.0546 0 0"/>
+    </joint>
+    <link name="base_plate_cx110l">
+        <parent link="world"/>
+        <visual>
+            <origin
+                xyz="0 0 0.0127"
+                rpy="0 0 0" />
+            <geometry>
+                <box size="1.016 1.016 0.0254" />
+            </geometry>
+            <material
+                name="">
+                <color
+                rgba="0.75294 0.75294 0.75294 1" />
+            </material>
+        </visual>
+        <collision>
+            <origin
+                xyz="0 0 0"
+                rpy="0 0 0" />
+            <geometry>
+                <box size="1.016 1.016 0.0254" />
+            </geometry>
+        </collision>
+        <xacro:default_inertial mass="1"/>
+    </link>
     <joint name="world2east_wall" type="fixed">
         <parent link="world"/>
@@ -47,21 +77,21 @@
         <visual>
             <origin
-                xyz="-0.7888 -0.7612 2.5"
-                rpy="0 0 0" />
-            <geometry>
-                <box size="3 0.1 5" />
-            </geometry>
-            <material
-                name="">
-                <color
-                rgba="0.75294 0.75294 0.75294 1" />
-            </material>
-        </visual>
-        <collision>
-            <origin
-                xyz="-0.7888 -0.7612 2.5"
-                rpy="0 0 0" />
-            <geometry>
-                <box size="3 0.1 5" />
+                xyz="-2.53 -0.81 2.5"
+                rpy="0 0 0" />
+            <geometry>
+                <box size="6.68 0.1 5" />
+            </geometry>
+            <material
+                name="">
+                <color
+                rgba="0.75294 0.75294 0.75294 1" />
+            </material>
+        </visual>
+        <collision>
+            <origin
+                xyz="-2.53 -0.81 2.5"
+                rpy="0 0 0" />
+            <geometry>
+                <box size="6.68 0.1 5" />
             </geometry>
         </collision>
@@ -76,21 +106,21 @@
         <visual>
             <origin
-                xyz="0.7612 0.9398 2.5"
-                rpy="0 0 0" />
-            <geometry>
-                <box size="0.1 3.302 5" />
-            </geometry>
-            <material
-                name="">
-                <color
-                rgba="0.75294 0.75294 0.75294 1" />
-            </material>
-        </visual>
-        <collision>
-            <origin
-                xyz="0.7612 0.9398 2.5"
-                rpy="0 0 0" />
-            <geometry>
-                <box size="0.1 3.302 5" />
+                xyz="0.810 1.717 2.5"
+                rpy="0 0 0" />
+            <geometry>
+                <box size="0.1 5.055 5" />
+            </geometry>
+            <material
+                name="">
+                <color
+                rgba="0.75294 0.75294 0.75294 1" />
+            </material>
+        </visual>
+        <collision>
+            <origin
+                xyz="0.810 1.717 2.5"
+                rpy="0 0 0" />
+            <geometry>
+                <box size="0.1 5.055 5" />
             </geometry>
         </collision>
@@ -105,21 +135,21 @@
         <visual>
             <origin
-                xyz="0 0 -0.05"
-                rpy="0 0 0" />
-            <geometry>
-                <box size="6 6 0.1" />
-            </geometry>
-            <material
-                name="">
-                <color
-                rgba="0.75294 0.75294 0.75294 1" />
-            </material>
-        </visual>
-        <collision>
-            <origin
-                xyz="0 0 -0.05"
-                rpy="0 0 0" />
-            <geometry>
-                <box size="6 6 0.1" />
+                xyz="-2.53 1.717 -0.063"
+                rpy="0 0 0" />
+            <geometry>
+                <box size="6.68 5.055 0.1" />
+            </geometry>
+            <material
+                name="">
+                <color
+                rgba="0.75294 0.75294 0.75294 1" />
+            </material>
+        </visual>
+        <collision>
+            <origin
+                xyz="-2.53 1.717 -0.063"
+                rpy="0 0 0" />
+            <geometry>
+                <box size="6.68 5.055 0.1" />
             </geometry>
         </collision>
@@ -134,21 +164,21 @@
         <visual>
             <origin
-                xyz="-0.7888 2.6392 2.5"
-                rpy="0 0 0" />
-            <geometry>
-                <box size="3 0.1 5" />
-            </geometry>
-            <material
-                name="">
-                <color
-                rgba="0.75294 0.75294 0.75294 0.2" />
-            </material>
-        </visual>
-        <collision>
-            <origin
-                xyz="-0.7888 2.6392 2.5"
-                rpy="0 0 0" />
-            <geometry>
-                <box size="3 0.1 5" />
+                xyz="-2.53 4.245 2.5"
+                rpy="0 0 0" />
+            <geometry>
+                <box size="6.68 0.1 5" />
+            </geometry>
+            <material
+                name="">
+                <color
+                rgba="0.75294 0.75294 0.75294 0.1" />
+            </material>
+        </visual>
+        <collision>
+            <origin
+                xyz="-2.53 4.245 2.5"
+                rpy="0 0 0" />
+            <geometry>
+                <box size="6.68 0.1 5" />
             </geometry>
         </collision>
@@ -163,21 +193,21 @@
         <visual>
             <origin
-                xyz="-2.3344 0.9398 2.5"
-                rpy="0 0 0" />
-            <geometry>
-                <box size="0.1 3.302 5" />
-            </geometry>
-            <material
-                name="">
-                <color
-                rgba="0.75294 0.75294 0.75294 0.2" />
-            </material>
-        </visual>
-        <collision>
-            <origin
-                xyz="-2.3344 0.9398 2.5"
-                rpy="0 0 0" />
-            <geometry>
-                <box size="0.1 3.302 5" />
+                xyz="-5.878 1.7175 2.5"
+                rpy="0 0 0" />
+            <geometry>
+                <box size="0.1 5.055 5" />
+            </geometry>
+            <material
+                name="">
+                <color
+                rgba="0.75294 0.75294 0.75294 0.1" />
+            </material>
+        </visual>
+        <collision>
+            <origin
+                xyz="-5.878 1.7175 2.5"
+                rpy="0 0 0" />
+            <geometry>
+                <box size="0.1 5.055 5" />
             </geometry>
         </collision>
