Commit message: the robot home position may be inaccurate

File: description/urdf/cx110l.urdf.xacro (robot description, xacro)
@@ -2,4 +2,5 @@
 <robot xmlns:xacro="http://wiki.ros.org/xacro" name="cx110l">
   <xacro:property name="robot_name" value="cx110l"/>
+  <xacro:property name="krnx_name" value="CX110L-BC01"/>
   <!-- Import cx110l macro -->
   <xacro:include filename="$(find khi2cpp_hw_description)/${robot_name}/urdf/${robot_name}_description.urdf.xacro"/>
