Commit message: corrections to urdf and added testing

File: cx110l/urdf/cx110l_description.urdf.xacro (robot description, xacro)
@@ -214,4 +214,10 @@
     <limit effort="1000.0" lower="${j6_lower_limit}" upper="${j6_upper_limit}" velocity="${j6_velocity_limit}"/>
   </joint>
+  <link name="tool0" />
+  <joint name="tool0_joint" type="fixed">
+    <parent link="link_6"/>
+    <child link="tool0"/>
+    <origin xyz="0 0 0" rpy="0 0 0"/>
+  </joint>
 </xacro:macro>
 </robot>
